File: PCB_DEV/GATE/gate.sch (EAGLE design)
At the start: 15 parts, among them K1 REED, K2 REED, K3 REED, U2 esp12

Commit message: w
Parts:
- added D1, D2, D3: 1N4148, diode:DIODE-SOD80C
- added J3Y, JY1, JY3: S8050, semicon-smd-ipc:NPN-TRANSISTOR_SOT23
- added R1, R12, R13, R2, R5, R6: 10k, resistor:R-EU_R0603
- added U$1: DC-DC-STEP-DOWN-LM2596, diy-modules:DC-DC-STEP-DOWN-LM2596
- added X1, X2, X3, X4: (no value), con-wago-500:W237-102
- DS18B20: device SparkFun-Connectors:CONN_03JST-PTH-VERT -> SparkFun-Connectors:CONN_03SCREW
- UART: device SparkFun-Connectors:CONN_04JST-PTH-VERT -> SparkFun-Connectors:CONN_04SCREW
Connections:
- new net 5V: U$1.OUT+
- new net GND1: K12.S, X2-1.KL
- new net GND2: K22.S, X3-1.KL
- new net GND3: K32.S, X4-1.KL
- new net N$1: K12.P, X2-2.KL
- new net N$13: JY3.B, R2.2, R5.2
- new net N$17: U$1.IN+, X1-2.KL
- new net N$2: K22.P, X3-2.KL
- new net N$3: K32.P, X4-2.KL
- new net N$4: D1.A, J3Y.C, K11.+
- new net N$5: D3.A, JY1.C, K31.+
- new net N$6: JY1.B, R12.2, R13.2
- new net N$7: J3Y.B, R1.2, R6.2
- new net N$9: D2.A, JY3.C, K21.+
- new net VCC: D1.C, D2.C, D3.C, K11.-, K21.-, K31.-
- net GND: now also J3Y.E, JY1.E, JY3.E, R13.1, R5.1, R6.1, U$1.IN-, U$1.OUT-, X1-1.KL
- net GPIO04: now also R1.1
- net GPIO05: now also R2.1
- net GPIO14: now also R12.1
Other:
- moved on the sheet: DS18B20, K1, K2, K3, R4, UART

Commit message: d
Parts:
- removed DS18B20: (no value), SparkFun-Connectors:CONN_03SCREW
- removed J3Y, JY1, JY3: S8050, semicon-smd-ipc:NPN-TRANSISTOR_SOT23
- removed R1, R12, R13, R2, R4, R5, R6: 10k, resistor:R-EU_R0603
- added CLOSE_S, OPEN_S: (no value), SparkFun-Connectors:CONN_023.5MM
- renumbered K1 to OPEN_R, K2 to STOP_R, K3 to CLOSE_R
Connections:
- removed net 5V: U$1.OUT+
- removed net N$13: JY3.B, R2.2, R5.2
- removed net N$4: D1.A, J3Y.C, OPEN_R1.+
- removed net N$5: CLOSE_R1.+, D3.A, JY1.C
- removed net N$6: JY1.B, R12.2, R13.2
- removed net N$7: J3Y.B, R1.2, R6.2
- removed net N$9: D2.A, JY3.C, STOP_R1.+
- removed net VCC: CLOSE_R1.-, D1.C, D2.C, D3.C, OPEN_R1.-, STOP_R1.-
- net 3V3: now also U$1.OUT+; no longer DS18B20.3, R4.2
- net GND: now also CLOSE_R1.+, CLOSE_S.1, D1.A, D2.A, D3.A, OPEN_R1.+, OPEN_S.1, STOP_R1.+; no longer DS18B20.1, J3Y.E, JY1.E, JY3.E, R13.1, R5.1, R6.1
- net GPIO04: now also D1.C, OPEN_R1.-; no longer R1.1
- net GPIO05: now also D2.C, STOP_R1.-; no longer R2.1
- net GPIO12: now also CLOSE_S.2; no longer DS18B20.2, R4.1
- net GPIO13: now also OPEN_S.2
- net GPIO14: now also CLOSE_R1.-, D3.C; no longer R12.1

Commit message: d
Parts:
- added J1: LDR-TH, kanflo:LDR-TH
- added R1: 10k, resistor:R-EU_R0603
Connections:
- net 3V3: now also J1.1
- net A0: now also J1.2, R1.1
- net GND: now also R1.2
Changed lines of the file:
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@@
 <part name="CLOSE_S" library="SparkFun-Connectors" library_urn="urn:adsk.eagle:library:513" deviceset="CONN_02" device="3.5MM" package3d_urn="urn:adsk.eagle:package:38050/1"/>
 <part name="OPEN_S" library="SparkFun-Connectors" library_urn="urn:adsk.eagle:library:513" deviceset="CONN_02" device="3.5MM" package3d_urn="urn:adsk.eagle:package:38050/1"/>
+<part name="J1" library="kanflo" deviceset="LDR" device="-TH"/>
+<part name="R1" library="resistor" library_urn="urn:adsk.eagle:library:348" deviceset="R-EU_" device="R0603" package3d_urn="urn:adsk.eagle:package:26057/1" value="10k"/>
 </parts>
 <sheets>
@@
 <attribute name="NAME" x="-30.48" y="3.048" size="1.778" layer="95" font="vector"/>
 </instance>
+<instance part="J1" gate="G$1" x="-93.98" y="0" smashed="yes">
+<attribute name="NAME" x="-97.89" y="-3.5014" size="1.778" layer="95"/>
+</instance>
+<instance part="R1" gate="G$1" x="-81.28" y="0" smashed="yes">
+<attribute name="NAME" x="-85.09" y="1.4986" size="1.778" layer="95"/>
+<attribute name="VALUE" x="-85.09" y="-3.302" size="1.778" layer="96"/>
+</instance>
 </instances>
 <busses>
@@
 <wire x1="-20.32" y1="-2.54" x2="-15.24" y2="-2.54" width="0.1524" layer="91"/>
 <label x="-15.24" y="-2.54" size="1.778" layer="95" xref="yes"/>
+</segment>
+<segment>
+<pinref part="R1" gate="G$1" pin="2"/>
+<wire x1="-76.2" y1="0" x2="-76.2" y2="10.16" width="0.1524" layer="91"/>
+<label x="-76.2" y="10.16" size="1.778" layer="95" xref="yes"/>
 </segment>
 </net>
@@
 <label x="83.82" y="2.54" size="1.778" layer="95" xref="yes"/>
 </segment>
+<segment>
+<pinref part="J1" gate="G$1" pin="1"/>
+<wire x1="-99.06" y1="0" x2="-101.6" y2="0" width="0.1524" layer="91"/>
+<wire x1="-101.6" y1="0" x2="-101.6" y2="5.08" width="0.1524" layer="91"/>
+<label x="-101.6" y="5.08" size="1.778" layer="95" rot="R90" xref="yes"/>
+</segment>
 </net>
 <net name="A0" class="0">
@@
 <label x="-5.08" y="60.96" size="1.778" layer="95" rot="R90" xref="yes"/>
 </segment>
-</net>
+<segment>
+<pinref part="J1" gate="G$1" pin="2"/>
+<pinref part="R1" gate="G$1" pin="1"/>
+<wire x1="-86.36" y1="0" x2="-88.9" y2="0" width="0.1524" layer="91"/>
+<wire x1="-86.36" y1="0" x2="-86.36" y2="7.62" width="0.1524" layer="91"/>
+<junction x="-86.36" y="0"/>
+<label x="-86.36" y="7.62" size="1.778" layer="95" xref="yes"/>
+</segment>
+</net>

Commit message: pcb done v1
Parts:
- renumbered J1 to LDR
Changed lines of the file:
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@@
 <part name="CLOSE_S" library="SparkFun-Connectors" library_urn="urn:adsk.eagle:library:513" deviceset="CONN_02" device="3.5MM" package3d_urn="urn:adsk.eagle:package:38050/1"/>
 <part name="OPEN_S" library="SparkFun-Connectors" library_urn="urn:adsk.eagle:library:513" deviceset="CONN_02" device="3.5MM" package3d_urn="urn:adsk.eagle:package:38050/1"/>
-<part name="J1" library="kanflo" deviceset="LDR" device="-TH"/>
+<part name="LDR" library="kanflo" deviceset="LDR" device="-TH"/>
 <part name="R1" library="resistor" library_urn="urn:adsk.eagle:library:348" deviceset="R-EU_" device="R0603" package3d_urn="urn:adsk.eagle:package:26057/1" value="10k"/>
 </parts>
@@
 <attribute name="NAME" x="-30.48" y="3.048" size="1.778" layer="95" font="vector"/>
 </instance>
-<instance part="J1" gate="G$1" x="-93.98" y="0" smashed="yes">
+<instance part="LDR" gate="G$1" x="-93.98" y="0" smashed="yes">
 <attribute name="NAME" x="-97.89" y="-3.5014" size="1.778" layer="95"/>
 </instance>
@@
 </segment>
 <segment>
-<pinref part="J1" gate="G$1" pin="1"/>
+<pinref part="LDR" gate="G$1" pin="1"/>
 <wire x1="-99.06" y1="0" x2="-101.6" y2="0" width="0.1524" layer="91"/>
 <wire x1="-101.6" y1="0" x2="-101.6" y2="5.08" width="0.1524" layer="91"/>
@@
 </segment>
 <segment>
-<pinref part="J1" gate="G$1" pin="2"/>
+<pinref part="LDR" gate="G$1" pin="2"/>
 <pinref part="R1" gate="G$1" pin="1"/>
 <wire x1="-86.36" y1="0" x2="-88.9" y2="0" width="0.1524" layer="91"/>

Commit message: v1
Parts:
- renumbered X1 to POWER, X2 to OPEN, X3 to STOP, X4 to CLOSE
Changed lines of the file:
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@@
 <part name="STOP_R" library="relay" library_urn="urn:adsk.eagle:library:339" deviceset="REED" device="" package3d_urn="urn:adsk.eagle:package:24297/1"/>
 <part name="CLOSE_R" library="relay" library_urn="urn:adsk.eagle:library:339" deviceset="REED" device="" package3d_urn="urn:adsk.eagle:package:24297/1"/>
-<part name="X1" library="con-wago-500" library_urn="urn:adsk.eagle:library:195" deviceset="W237-102" device="" package3d_urn="urn:adsk.eagle:package:10688/1"/>
+<part name="POWER" library="con-wago-500" library_urn="urn:adsk.eagle:library:195" deviceset="W237-102" device="" package3d_urn="urn:adsk.eagle:package:10688/1"/>
 <part name="U$1" library="diy-modules" deviceset="DC-DC-STEP-DOWN-LM2596" device=""/>
-<part name="X2" library="con-wago-500" library_urn="urn:adsk.eagle:library:195" deviceset="W237-102" device="" package3d_urn="urn:adsk.eagle:package:10688/1"/>
-<part name="X3" library="con-wago-500" library_urn="urn:adsk.eagle:library:195" deviceset="W237-102" device="" package3d_urn="urn:adsk.eagle:package:10688/1"/>
-<part name="X4" library="con-wago-500" library_urn="urn:adsk.eagle:library:195" deviceset="W237-102" device="" package3d_urn="urn:adsk.eagle:package:10688/1"/>
+<part name="OPEN" library="con-wago-500" library_urn="urn:adsk.eagle:library:195" deviceset="W237-102" device="" package3d_urn="urn:adsk.eagle:package:10688/1"/>
+<part name="STOP" library="con-wago-500" library_urn="urn:adsk.eagle:library:195" deviceset="W237-102" device="" package3d_urn="urn:adsk.eagle:package:10688/1"/>
+<part name="CLOSE" library="con-wago-500" library_urn="urn:adsk.eagle:library:195" deviceset="W237-102" device="" package3d_urn="urn:adsk.eagle:package:10688/1"/>
 <part name="D1" library="diode" library_urn="urn:adsk.eagle:library:210" deviceset="DIODE-" device="SOD80C" package3d_urn="urn:adsk.eagle:package:43405/2" value="1N4148"/>
 <part name="D2" library="diode" library_urn="urn:adsk.eagle:library:210" deviceset="DIODE-" device="SOD80C" package3d_urn="urn:adsk.eagle:package:43405/2" value="1N4148"/>
@@
 <attribute name="PART" x="92.71" y="63.5" size="1.778" layer="95"/>
 </instance>
-<instance part="X1" gate="-1" x="27.94" y="-7.62" smashed="yes">
+<instance part="POWER" gate="-1" x="27.94" y="-7.62" smashed="yes">
 <attribute name="NAME" x="27.94" y="-6.731" size="1.778" layer="95" rot="R180"/>
 </instance>
-<instance part="X1" gate="-2" x="27.94" y="2.54" smashed="yes">
+<instance part="POWER" gate="-2" x="27.94" y="2.54" smashed="yes">
 <attribute name="VALUE" x="25.4" y="-1.143" size="1.778" layer="96"/>
 <attribute name="NAME" x="27.94" y="3.429" size="1.778" layer="95" rot="R180"/>
@@
 <attribute name="VALUE" x="43.18" y="10.16" size="1.778" layer="96"/>
 </instance>
-<instance part="X2" gate="-1" x="43.18" y="137.16" smashed="yes" rot="R180">
+<instance part="OPEN" gate="-1" x="43.18" y="137.16" smashed="yes" rot="R180">
 <attribute name="NAME" x="43.18" y="136.271" size="1.778" layer="95"/>
 </instance>
-<instance part="X2" gate="-2" x="43.18" y="127" smashed="yes" rot="R180">
+<instance part="OPEN" gate="-2" x="43.18" y="127" smashed="yes" rot="R180">
 <attribute name="VALUE" x="45.72" y="130.683" size="1.778" layer="96" rot="R180"/>
 <attribute name="NAME" x="43.18" y="126.111" size="1.778" layer="95"/>
 </instance>
-<instance part="X3" gate="-1" x="43.18" y="111.76" smashed="yes" rot="R180">
+<instance part="STOP" gate="-1" x="43.18" y="111.76" smashed="yes" rot="R180">
 <attribute name="NAME" x="43.18" y="110.871" size="1.778" layer="95"/>
 </instance>
-<instance part="X3" gate="-2" x="43.18" y="101.6" smashed="yes" rot="R180">
+<instance part="STOP" gate="-2" x="43.18" y="101.6" smashed="yes" rot="R180">
 <attribute name="VALUE" x="45.72" y="105.283" size="1.778" layer="96" rot="R180"/>
 <attribute name="NAME" x="43.18" y="100.711" size="1.778" layer="95"/>
 </instance>
-<instance part="X4" gate="-1" x="45.72" y="93.98" smashed="yes" rot="R180">
+<instance part="CLOSE" gate="-1" x="45.72" y="93.98" smashed="yes" rot="R180">
 <attribute name="NAME" x="45.72" y="93.091" size="1.778" layer="95"/>
 </instance>
-<instance part="X4" gate="-2" x="45.72" y="83.82" smashed="yes" rot="R180">
+<instance part="CLOSE" gate="-2" x="45.72" y="83.82" smashed="yes" rot="R180">
 <attribute name="VALUE" x="48.26" y="87.503" size="1.778" layer="96" rot="R180"/>
 <attribute name="NAME" x="45.72" y="82.931" size="1.778" layer="95"/>
@@
 <segment>
 <pinref part="U$1" gate="G$1" pin="IN-"/>
-<pinref part="X1" gate="-1" pin="KL"/>
+<pinref part="POWER" gate="-1" pin="KL"/>
 <wire x1="33.02" y1="-7.62" x2="38.1" y2="-7.62" width="0.1524" layer="91"/>
 </segment>
@@
 <segment>
 <pinref part="U$1" gate="G$1" pin="IN+"/>
-<pinref part="X1" gate="-2" pin="KL"/>
+<pinref part="POWER" gate="-2" pin="KL"/>
 <wire x1="33.02" y1="2.54" x2="38.1" y2="2.54" width="0.1524" layer="91"/>
 </segment>
@@
 <net name="GND1" class="0">
 <segment>
-<pinref part="X2" gate="-1" pin="KL"/>
+<pinref part="OPEN" gate="-1" pin="KL"/>
 <wire x1="38.1" y1="137.16" x2="22.86" y2="137.16" width="0.1524" layer="91"/>
 <pinref part="OPEN_R" gate="2" pin="S"/>
@@
 <net name="N$1" class="0">
 <segment>
-<pinref part="X2" gate="-2" pin="KL"/>
+<pinref part="OPEN" gate="-2" pin="KL"/>
 <pinref part="OPEN_R" gate="2" pin="P"/>
 <wire x1="22.86" y1="127" x2="38.1" y2="127" width="0.1524" layer="91"/>
@@
 <net name="GND2" class="0">
 <segment>
-<pinref part="X3" gate="-1" pin="KL"/>
+<pinref part="STOP" gate="-1" pin="KL"/>
 <wire x1="38.1" y1="111.76" x2="33.02" y2="111.76" width="0.1524" layer="91"/>
 <pinref part="STOP_R" gate="2" pin="S"/>
@@
 <net name="N$2" class="0">
 <segment>
-<pinref part="X3" gate="-2" pin="KL"/>
+<pinref part="STOP" gate="-2" pin="KL"/>
 <wire x1="38.1" y1="101.6" x2="33.02" y2="101.6" width="0.1524" layer="91"/>
 <pinref part="STOP_R" gate="2" pin="P"/>
@@
 <net name="GND3" class="0">
 <segment>
-<pinref part="X4" gate="-1" pin="KL"/>
+<pinref part="CLOSE" gate="-1" pin="KL"/>
 <pinref part="CLOSE_R" gate="2" pin="S"/>
 <wire x1="22.86" y1="93.98" x2="40.64" y2="93.98" width="0.1524" layer="91"/>
@@
 <net name="N$3" class="0">
 <segment>
-<pinref part="X4" gate="-2" pin="KL"/>
+<pinref part="CLOSE" gate="-2" pin="KL"/>
 <pinref part="CLOSE_R" gate="2" pin="P"/>
 <wire x1="22.86" y1="83.82" x2="40.64" y2="83.82" width="0.1524" layer="91"/>

Commit message: gate
Connections:
- net 3V3: now also LDR.2; no longer LDR.1
- net A0: now also LDR.1; no longer LDR.2
Other:
- moved on the sheet: LDR
Changed lines of the file:
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@@
 <attribute name="NAME" x="-30.48" y="3.048" size="1.778" layer="95" font="vector"/>
 </instance>
-<instance part="LDR" gate="G$1" x="-93.98" y="0" smashed="yes">
-<attribute name="NAME" x="-97.89" y="-3.5014" size="1.778" layer="95"/>
+<instance part="LDR" gate="G$1" x="-93.98" y="0" smashed="yes" rot="R180">
+<attribute name="NAME" x="-90.07" y="3.5014" size="1.778" layer="95" rot="R180"/>
 </instance>
 <instance part="R1" gate="G$1" x="-81.28" y="0" smashed="yes">
@@
 </segment>
 <segment>
-<pinref part="LDR" gate="G$1" pin="1"/>
-<wire x1="-99.06" y1="0" x2="-101.6" y2="0" width="0.1524" layer="91"/>
 <wire x1="-101.6" y1="0" x2="-101.6" y2="5.08" width="0.1524" layer="91"/>
 <label x="-101.6" y="5.08" size="1.778" layer="95" rot="R90" xref="yes"/>
+<pinref part="LDR" gate="G$1" pin="2"/>
+<wire x1="-99.06" y1="0" x2="-101.6" y2="0" width="0.1524" layer="91"/>
 </segment>
 </net>
@@
 </segment>
 <segment>
-<pinref part="LDR" gate="G$1" pin="2"/>
 <pinref part="R1" gate="G$1" pin="1"/>
-<wire x1="-86.36" y1="0" x2="-88.9" y2="0" width="0.1524" layer="91"/>
 <wire x1="-86.36" y1="0" x2="-86.36" y2="7.62" width="0.1524" layer="91"/>
+<label x="-86.36" y="7.62" size="1.778" layer="95" xref="yes"/>
+<pinref part="LDR" gate="G$1" pin="1"/>
+<wire x1="-88.9" y1="0" x2="-86.36" y2="0" width="0.1524" layer="91"/>
 <junction x="-86.36" y="0"/>
-<label x="-86.36" y="7.62" size="1.778" layer="95" xref="yes"/>
-</segment>
-</net>
+</segment>
+</net>
