File: PCB_DEV/GATE/gate.brd (EAGLE design)
At the start: 45.5 x 78.4 mm, 32 parts, among them J3Y S8050, K1 REED, K2 REED, K3 REED, U2 esp12

Commit message: d
Parts:
- removed DS18B20: (no value), SparkFun-Connectors:SCREWTERMINAL-3.5MM-3
- removed J3Y, JY1, JY3: S8050, semicon-smd-ipc:SOT23
- removed R1, R12, R13, R2, R4, R5, R6: 10k, resistor:R0603
- added CLOSE_S, OPEN_S: (no value), SparkFun-Connectors:SCREWTERMINAL-3.5MM-2
- moved D3 69.6 mm to (22.8, 9.11), turned to 180 degrees
- moved D1 41.3 mm to (22.6, 23.9), turned to 180 degrees
- moved D2 27.7 mm to (22.8, 12.6), turned to 180 degrees
- moved UART 11.2 mm to (40.8, 42.9), turned to 270 degrees
- renumbered K1 to OPEN_R, K2 to STOP_R, K3 to CLOSE_R
Connections:
- removed net 5V: U$1.OUT+
- removed net N$13: JY3.1, R2.2, R5.2
- removed net N$4: D1.A, J3Y.3, OPEN_R.3
- removed net N$5: CLOSE_R.3, D3.A, JY1.3
- removed net N$6: JY1.1, R12.2, R13.2
- removed net N$7: J3Y.1, R1.2, R6.2
- removed net N$9: D2.A, JY3.3, STOP_R.3
- removed net VCC: CLOSE_R.5, D1.C, D2.C, D3.C, OPEN_R.5, STOP_R.5
- net 3V3: now also U$1.OUT+; no longer DS18B20.3, R4.2
- net GND: now also CLOSE_R.3, CLOSE_S.1, D1.A, D2.A, D3.A, OPEN_R.3, OPEN_S.1, STOP_R.3; no longer DS18B20.1, J3Y.2, JY1.2, JY3.2, R13.1, R5.1, R6.1
- net GPIO04: now also D1.C, OPEN_R.5; no longer R1.1
- net GPIO05: now also D2.C, STOP_R.5; no longer R2.1
- net GPIO12: now also CLOSE_S.2; no longer DS18B20.2, R4.1
- net GPIO13: now also OPEN_S.2
- net GPIO14: now also CLOSE_R.5, D3.C; no longer R12.1

Commit message: d
Parts:
- added J1: LDR-TH, kanflo:1X02
- added R1: 10k, resistor:R0603
- moved R7 4.33 mm to (9.82, 33.3)
- moved R3 4.31 mm to (13.3, 33.3)
- moved R9 4.04 mm to (16.7, 33.3)
- moved X2 1.39 mm to (3.96, 26.2)
- moved R8 1.01 mm to (22.4, 33.4)
- moved X3 0.79 mm to (3.95, 15.7)
Connections:
- net 3V3: now also J1.1
- net A0: now also J1.2, R1.1
- net GND: now also R1.2

Commit message: pcb done v1
Parts:
- removed J1: LDR-TH, kanflo:1X02
- added LDR: LDR-TH, kanflo:1X02
Connections:
- net 3V3: now also LDR.1; no longer J1.1
- net A0: now also LDR.2; no longer J1.2
Routing:
- net GND: track 0.00 -> 221.2 mm, vias 0 -> 2
- net 3V3: track 0.00 -> 75.7 mm, vias 0 -> 1
- net GPIO05: track 0.00 -> 63.9 mm, vias 0 -> 1
- net GPIO04: track 0.00 -> 60.6 mm
- net RX: track 0.00 -> 55.7 mm
- net TX: track 0.00 -> 43.1 mm
- net GPIO0: track 0.00 -> 41.5 mm
- net GPIO14: track 0.00 -> 41.0 mm, vias 0 -> 1
- net GPIO13: track 0.00 -> 38.8 mm, vias 0 -> 1
- net GPIO12: track 0.00 -> 30.9 mm, vias 0 -> 1
- net GND1: track 0.00 -> 27.0 mm
- net GND2: track 0.00 -> 26.7 mm
- net GND3: track 0.00 -> 26.4 mm
- net RESET: track 0.00 -> 26.2 mm
- net A0: track 0.00 -> 13.9 mm
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Other:
- board text added: "BH GATE v1"

Commit message: v1
Parts:
- removed X2, X3: (no value), con-wago-500:W237-102
- added OPEN, STOP: (no value), con-wago-500:W237-102
- moved R8 4.72 mm to (27.1, 33.4), turned to 180 degrees
- moved R3 0.72 mm to (12.6, 33.4)
- moved R9 0.50 mm to (16.2, 33.4)
- moved CLOSE_R 0.15 mm to (32.9, 2.54)
- moved OPEN_R 0.15 mm to (32.9, 25.4)
- moved STOP_R 0.15 mm to (32.9, 14.0)
- moved R7 0.09 mm to (9.82, 33.4)
- moved D1 0.09 mm to (22.7, 23.9)
- moved OPEN_S 0.09 mm to (40.6, 4.06)
- moved D3 0.08 mm to (22.7, 9.11)
- renumbered X1 to POWER, X4 to CLOSE
Connections:
- net GND1: now also OPEN.1; no longer X2.1
- net GND2: now also STOP.1; no longer X3.1
- net N$1: now also OPEN.2; no longer X2.2
- net N$2: now also STOP.2; no longer X3.2
Routing:
- net GPIO0: track 41.5 -> 36.3 mm
- net 3V3: track 75.7 -> 79.2 mm
- net GPIO05: track 63.9 -> 62.8 mm
- net RX: track 55.7 -> 54.8 mm
- net A0: track 13.9 -> 13.1 mm
- net ADC: track 7.32 -> 6.49 mm
- net CH_PD: track 6.01 -> 5.50 mm

Commit message: gate
Parts:
- moved FLASH 10.2 mm to (40.5, 43.0), turned to 0 degrees
- moved RESET 9.66 mm to (40.5, 37.7), turned to 0 degrees
- moved UART 9.39 mm to (40.3, 33.5)
- moved R7 6.39 mm to (16.2, 33.4)
- moved R9 4.94 mm to (21.1, 33.4)
- moved R11 3.70 mm to (28.2, 54.8), turned to 270 degrees
- moved R10 2.77 mm to (32.0, 33.4), turned to 90 degrees
- moved R1 2.02 mm to (5.63, 33.6), turned to 270 degrees
- moved POWER 1.46 mm to (39.2, 50.9), turned to 90 degrees
- moved R3 1.40 mm to (11.2, 33.5)
- moved D1 0.74 mm to (22.3, 23.3), flipped to the bottom, turned to 0 degrees
- moved D2 0.62 mm to (22.3, 12.1), flipped to the bottom, turned to 0 degrees
- moved R8 0.50 mm to (26.6, 33.4), turned to 90 degrees
- moved D3 0.39 mm to (22.3, 9.24), flipped to the bottom, turned to 0 degrees
- moved LDR 0.07 mm to (1.52, 34.5)
Connections:
- net 3V3: now also LDR.2; no longer LDR.1
- net A0: now also LDR.1; no longer LDR.2
Routing:
- net GPIO12: track 30.9 -> 73.1 mm, vias 1 -> 0
- net GPIO0: track 36.3 -> 68.8 mm
- net GPIO04: track 60.5 -> 38.2 mm, vias 0 -> 1
- net GND: track 221.6 -> 202.9 mm, vias 2 -> 0
- net GPIO05: track 62.8 -> 51.3 mm
- net RESET: track 26.2 -> 36.9 mm, vias 0 -> 2
- net TX: track 43.0 -> 53.4 mm
- net RX: track 54.8 -> 44.6 mm, vias 0 -> 1
- net GPIO13: track 38.7 -> 45.8 mm, vias 1 -> 0
- net N$17: track 11.8 -> 6.18 mm
- net GPIO14: track 40.9 -> 46.0 mm
- net CH_PD: track 5.50 -> 10.3 mm
- net GPIO15: track 5.52 -> 8.79 mm
- net ADC: track 6.49 -> 8.97 mm
- net A0: track 13.1 -> 10.9 mm
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- added copper zone on layer 1, net GND
- added copper zone on layer 16, net GND

Commit message: V1
V1
Parts:
- renumbered CLOSE to RELAY_3, CLOSE_R to RELAY_3_C, OPEN to RELAY_1, OPEN_R to RELAY_1_C, STOP to RELAY_2, STOP_R to RELAY_2_C
